File: 4067/4067.kicad_pcb (KiCad board)
At the start: 2 copper layers, 45.1 x 49.3 mm, 9 parts, among them J1 Conn_02x16_Odd_Even, J2 Conn_02x04_Odd_Even, J3 Conn_02x01, J4 Conn_02x01, J5 VCC, J6 GND, U1 CD4067

Commit message: new routing
Parts:
- moved J1 5.46 mm to (128.9, 61.8)
Routing:
- net GND: track 0.00 -> 113.9 mm, vias 0 -> 4
- net Net-(J1-Pin_21): track 29.6 -> 113.5 mm
- net Net-(J1-Pin_23): track 29.6 -> 112.2 mm
- net Net-(J1-Pin_19): track 29.6 -> 94.2 mm
- net Net-(J1-Pin_25): track 29.6 -> 93.5 mm
- net Net-(J1-Pin_17): track 29.6 -> 83.4 mm
- net Net-(J1-Pin_15): track 15.3 -> 42.6 mm
- net Net-(J1-Pin_13): track 18.9 -> 39.7 mm
- net Net-(J1-Pin_3): track 25.1 -> 39.8 mm
- net Net-(J1-Pin_7): track 31.1 -> 44.6 mm
- net Net-(J1-Pin_10): track 28.5 -> 15.8 mm
- net Net-(J2-Pin_5): track 24.9 -> 37.3 mm
- net VCC: track 0.00 -> 11.8 mm, vias 0 -> 1
- net Net-(J1-Pin_11): track 25.1 -> 16.5 mm, vias 0 -> 1
- net Net-(J1-Pin_5): track 34.6 -> 42.2 mm
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Other:
- board size 45.1 x 49.3 mm -> 69.8 x 81.7 mm

Commit message: new routing
Other:
- board size 69.8 x 81.7 mm -> 53.6 x 56.8 mm
Changed lines of the file:
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@@
 	)
 	(gr_rect
-		(start 110.5 41.3)
-		(end 180.3 123)
+		(start 121.6 54.3)
+		(end 175.2 111.1)
 		(stroke
 			(width 0.05)

Commit message: remove unused tracks
Routing:
- net Net-(J1-Pin_25): track 93.5 -> 74.0 mm
- net Net-(J1-Pin_23): track 112.2 -> 92.7 mm
- net Net-(J1-Pin_21): track 113.5 -> 94.0 mm
- net Net-(J1-Pin_19): track 94.2 -> 74.7 mm
- net Net-(J1-Pin_17): track 83.4 -> 78.2 mm
- net Net-(J3-Pin_1): track 30.5 -> 29.4 mm
- net Net-(J1-Pin_29): track 35.1 -> 34.4 mm
Changed lines of the file:
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@@
-	)
-	(segment
-		(start 168.465 64.3)
-		(end 150.995 64.3)
-		(width 0.4)
-		(layer "B.Cu")
-		(net 3)
-	)
-	(segment
-		(start 150.995 64.3)
-		(end 146.1329 64.3)
-		(width 0.4)
-		(layer "B.Cu")
-		(net 3)
 	)
 	(segment
 		(start 146.1329 64.3)
-		(end 145.02 64.3)
+		(end 168.465 64.3)
 		(width 0.4)
 		(layer "B.Cu")
@@
 	)
 	(segment
-		(start 157.92 74.26)
-		(end 144.119 88.061)
-		(width 0.4)
-		(layer "F.Cu")
-		(net 11)
-	)
-	(segment
 		(start 131.44 87.16)
 		(end 128.9 87.16)
@@
 	(segment
 		(start 157.92 79.34)
-		(end 144.119 93.141)
-		(width 0.4)
-		(layer "F.Cu")
-		(net 12)
-	)
-	(segment
-		(start 157.92 79.34)
 		(end 157.92 79.8681)
 		(width 0.4)
@@
 	)
 	(segment
-		(start 157.92 71.72)
-		(end 144.119 85.521)
-		(width 0.4)
-		(layer "F.Cu")
-		(net 13)
-	)
-	(segment
 		(start 128.9 84.62)
 		(end 124.5969 80.3169)
@@
 	)
 	(segment
-		(start 157.92 76.8)
-		(end 144.119 90.601)
-		(width 0.4)
-		(layer "F.Cu")
-		(net 14)
-	)
-	(segment
 		(start 163.1444 107.3)
 		(end 134.4002 107.3)
@@
 	(segment
 		(start 143.8782 95.9218)
-		(end 144.119 95.681)
-		(width 0.4)
-		(layer "F.Cu")
-		(net 17)
-	)
-	(segment
-		(start 157.92 81.88)
-		(end 144.119 95.681)
+		(end 157.92 81.88)
 		(width 0.4)
 		(layer "F.Cu")
@@
 	(segment
 		(start 145.5441 96.7959)
-		(end 145.02 97.32)
-		(width 0.4)
-		(layer "F.Cu")
-		(net 18)
-	)
-	(segment
-		(start 145.5441 96.7959)
 		(end 131.9641 96.7959)
 		(width 0.4)
@@
 	(segment
 		(start 128.9 66.84)
-		(end 130.3216 66.84)
-		(width 0.4)
-		(layer "B.Cu")
-		(net 19)
-	)
-	(segment
-		(start 130.3216 66.84)
 		(end 131.44 66.84)
 		(width 0.4)
@@
 	)
 	(segment
-		(start 147.8446 79.2554)
-		(end 144.119 82.981)
-		(width 0.4)
-		(layer "F.Cu")
-		(net 21)
-	)
-	(segment
 		(start 125.3428 78.5228)
 		(end 125.3428 59.8221)
@@
 	)
 	(segment
-		(start 151.5701 75.5299)
-		(end 147.8446 79.2554)
+		(start 147.8446 79.2554)
+		(end 157.92 69.18)
 		(width 0.4)
 		(layer "F.Cu")
@@
 		(width 0.4)
 		(layer "F.Cu")
-		(net 21)
-	)
-	(segment
-		(start 157.92 69.18)
-		(end 151.5701 75.5299)
-		(width 0.4)
-		(layer "F.Cu")
