File: multistate filter/multistate filter.kicad_pcb (KiCad board)
At the start: 2 copper layers, 60 x 60 mm, 14 parts, among them J1 VCC, J2 GND, J3 IN, J4 HP, J5 BP, J6 LP, U1 4069

Commit message: multistate filter with potentiometer
Parts:
- added RV2: 100k, Potentiometer_THT:Potentiometer_Alps_RK163_Single_Horizontal, F.Cu at (113.0, 91.0)
Routing:
- net Net-(C1-Pad2): track 127.4 -> 33.4 mm
- net Net-(R3-Pad2): track 15.2 -> 64.2 mm
- net Net-(J5-Pin_1): track 51.9 -> 87.8 mm
Other:
- board size 60 x 60 mm -> 60 x 63 mm

Commit message: multistate filter v2
Routing:
- net Net-(C1-Pad2): track 33.4 -> 46.5 mm, vias 0 -> 2
Changed lines of the file:
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@@
+	)
+	(segment
+		(start 130 59.399)
+		(end 130 76.25)
+		(width 0.8)
+		(layer "F.Cu")
+		(net 1)
+	)
+	(segment
+		(start 130 76.25)
+		(end 124.5 81.75)
+		(width 0.8)
+		(layer "F.Cu")
+		(net 1)
+	)
+	(via
+		(at 130 59.399)
+		(size 1)
+		(drill 0.8)
+		(layers "F.Cu" "B.Cu")
+		(net 1)
+	)
+	(via
+		(at 124.5 81.75)
+		(size 1)
+		(drill 0.8)
+		(layers "F.Cu" "B.Cu")
+		(net 1)
 	)
 	(segment
 		(start 122.08 81.75)
-		(end 127.17 81.75)
+		(end 124.5 81.75)
 		(width 0.8)
 		(layer "B.Cu")
@@
 	)
 	(segment
-		(start 120.479 83.351)
-		(end 111.256844 83.351)
+		(start 130 59.399)
+		(end 123.511 59.399)
+		(width 0.8)
+		(layer "B.Cu")
+		(net 1)
+	)
+	(segment
+		(start 124.5 81.75)
+		(end 127.17 81.75)
 		(width 0.8)
 		(layer "B.Cu")
@@
 	(segment
 		(start 135.649 59.399)
-		(end 123.511 59.399)
-		(width 0.8)
-		(layer "B.Cu")
-		(net 1)
-	)
-	(segment
-		(start 122.08 81.75)
-		(end 120.479 83.351)
+		(end 130 59.399)
 		(width 0.8)
 		(layer "B.Cu")
@@
 	)
 	(segment
-		(start 139.475 55)
-		(end 142.015 55)
-		(width 0.4)
+		(start 139.475 60.725)
+		(end 139.75 61)
+		(width 0.8)
 		(layer "B.Cu")
 		(net 2)
@@
 		(start 139.475 55)
 		(end 139.475 60.725)
-		(width 0.4)
+		(width 0.8)
 		(layer "B.Cu")
 		(net 2)
@@
 	)
 	(segment
-		(start 139.475 60.725)
-		(end 139.75 61)
-		(width 0.4)
+		(start 139.475 55)
+		(end 142.015 55)
+		(width 0.8)
 		(layer "B.Cu")
 		(net 2)
